File: rev_c/bus_sonar10.kicad_pcb (KiCad board)
At the start: 2 copper layers, 100 x 50 mm, 39 parts, among them J1 TERMINATE_JUMPER, SW1 MJTP1243, U1 74HCT08, U2 LM2940, U3 MCP2562, U4 ATMEGA328_DIP28, U5 74HCT32, X1 16MHz

Commit message: Wrapped up Rev. C
Parts:
- added R10: 100K, bus_sonar10:Pin_Header_Straight_1x09, F.Cu at (196.8, 120.0)
- moved SW1 11.4 mm to (196.2, 137.2)
Connections:
- net +5V renamed VCC
Routing:
- net GND: track 142.7 -> 192.5 mm, vias 4 -> 8
- net /D12: track 23.4 -> 54.5 mm
- net Net-(N3-Pad3): track 38.8 -> 68.3 mm
- net Net-(N4-Pad11): track 61.9 -> 90.9 mm
- net Net-(N3-Pad11): track 34.1 -> 61.6 mm
- net Net-(N4-Pad3): track 69.0 -> 95.5 mm
- net Net-(N3-Pad35): track 14.9 -> 34.8 mm
- net /~RESET: track 57.6 -> 77.0 mm
- net Net-(N4-Pad35): track 35.2 -> 54.1 mm
- net Net-(N4-Pad27): track 45.0 -> 61.3 mm
- net Net-(C10-Pad1): track 36.3 -> 39.9 mm
- net /D13: track 31.4 -> 28.1 mm
- net /D10: track 41.5 -> 39.3 mm
- net /D3: track 51.9 -> 50.1 mm
- net /D8: track 29.3 -> 30.4 mm
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Other:
- board text added: "BUS_SONAR10 REV. C 17OCT2014 (c) GRAMLICH"
- board text removed: "BUS_SONAR10 REV. B 3OCT2014 (c) GRAMLICH"
